File: fm_tuner.sch (KiCad schematic (older format))
At the start: 17 parts, among them IC1 ATMEGA328P-A, J1 ISP_Header, P2 USB_B, SW1 SW_PUSH, U1 16x2_LCD, U2 si4713_module

Commit message: added first pass of routes to the board
Parts:
- C1, C2: footprint Capacitors_SMD:C_0201 -> Capacitors_SMD:C_0805_HandSoldering
- R1, R2, R3, R4, R5: footprint Resistors_SMD:R_0201 -> Resistors_SMD:R_0805_HandSoldering
Changed lines of the file:
@@
 F 0 "R1" V 4630 3300 50  0000 C CNN
 F 1 "10K" V 4550 3300 50  0000 C CNN
-F 2 "Resistors_SMD:R_0201" V 4480 3300 30  0001 C CNN
+F 2 "Resistors_SMD:R_0805_HandSoldering" V 4480 3300 30  0001 C CNN
 F 3 "" H 4550 3300 30  0000 C CNN
 	1    4550 3300
@@
 F 0 "R2" V 6980 2350 50  0000 C CNN
 F 1 "10K" V 6900 2350 50  0000 C CNN
-F 2 "Resistors_SMD:R_0201" V 6830 2350 30  0001 C CNN
+F 2 "Resistors_SMD:R_0805_HandSoldering" V 6830 2350 30  0001 C CNN
 F 3 "" H 6900 2350 30  0000 C CNN
 	1    6900 2350
@@
 F 0 "R3" V 7430 3850 50  0000 C CNN
 F 1 "10K" V 7350 3850 50  0000 C CNN
-F 2 "Resistors_SMD:R_0201" V 7280 3850 30  0001 C CNN
+F 2 "Resistors_SMD:R_0805_HandSoldering" V 7280 3850 30  0001 C CNN
 F 3 "" H 7350 3850 30  0000 C CNN
 	1    7350 3850
@@
 F 0 "C2" H 7925 2000 50  0000 L CNN
 F 1 "100n" H 7925 1800 50  0000 L CNN
-F 2 "Capacitors_SMD:C_0201" H 7938 1750 30  0001 C CNN
+F 2 "Capacitors_SMD:C_0805_HandSoldering" H 7938 1750 30  0001 C CNN
 F 3 "" H 7900 1900 60  0000 C CNN
 	1    7900 1900
@@
 F 0 "C1" H 7925 1700 50  0000 L CNN
 F 1 "100n" H 7925 1500 50  0000 L CNN
-F 2 "Capacitors_SMD:C_0201" H 7938 1450 30  0001 C CNN
+F 2 "Capacitors_SMD:C_0805_HandSoldering" H 7938 1450 30  0001 C CNN
 F 3 "" H 7900 1600 60  0000 C CNN
 	1    7900 1600
@@
 F 0 "R4" V 4930 2300 50  0000 C CNN
 F 1 "R" V 4850 2300 50  0000 C CNN
-F 2 "Resistors_SMD:R_0201" V 4780 2300 30  0001 C CNN
+F 2 "Resistors_SMD:R_0805_HandSoldering" V 4780 2300 30  0001 C CNN
 F 3 "" H 4850 2300 30  0000 C CNN
 	1    4850 2300
@@
 F 0 "R5" V 8980 1950 50  0000 C CNN
 F 1 "R" V 8900 1950 50  0000 C CNN
-F 2 "Resistors_SMD:R_0201" V 8830 1950 30  0001 C CNN
+F 2 "Resistors_SMD:R_0805_HandSoldering" V 8830 1950 30  0001 C CNN
 F 3 "" H 8900 1950 30  0000 C CNN
 	1    8900 1950

Commit message: added a new footprint for LCD with no silkscreen outline of the screen replaced LCD footprint on board wiht new one changed pour clearance
Parts:
- U1: footprint fm_tuner:16x2_LCD -> fm_tuner:16x2_LCD_noscreen
Changed lines of the file:
@@
 F 0 "U1" H 5750 4850 60  0000 C CNN
 F 1 "16x2_LCD" H 5900 5600 60  0000 C CNN
-F 2 "fm_tuner:16x2_LCD" H 5750 4850 60  0001 C CNN
+F 2 "fm_tuner:16x2_LCD_noscreen" H 5750 4850 60  0001 C CNN
 F 3 "" H 5750 4850 60  0000 C CNN
 	1    6000 5300
