File: fm_tuner.kicad_pcb (KiCad board)
At the start: 2 copper layers, 49 x 68.6 mm, 17 parts, among them IC1 ATMEGA328P-A, J1 ISP_Header, P2 USB_B, SW1 SW_PUSH, U1 16x2_LCD, U2 si4713_module

Commit message: remade gerbers
Parts:
- moved R5 6.04 mm to (28.7, 24.4)
- moved D2 5.36 mm to (20.6, 23.6)
- moved D1 4.93 mm to (20.6, 30.0)
- moved P2 3.34 mm to (21.1, 38.4)
Routing:
- net VCC: track 87.5 -> 64.9 mm, vias 3 -> 4
- net Net-(D1-Pad2): track 13.8 -> 10.3 mm
- removed copper zone on B.Cu, net VCC
Other:
- board size 49 x 68.6 mm -> 47 x 68.6 mm
Changed lines of the file:
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@@
   (general
     (links 57)
-    (no_connects 1)
-    (area 13.132999 13.132999 62.305001 81.863001)
+    (no_connects 7)
+    (area -64.790201 13.132999 62.305001 81.863001)
     (thickness 1.6)
     (drawings 8)
-    (tracks 174)
+    (tracks 176)
     (zones 0)
     (modules 17)
@@
   (layers
     (0 F.Cu signal)
-    (31 B.Cu signal hide)
+    (31 B.Cu signal)
     (32 B.Adhes user)
     (33 F.Adhes user)
@@
   )
   (module Connect:USB_Micro-B (layer F.Cu)
-    (at 17.78 38.862 270)
+    (at 21.082 38.354 270)
     (descr "Micro USB Type B Receptacle")
     (tags "USB USB_B USB_micro USB_OTG")
@@
   )
   (module Diodes_SMD:SMA_Standard (layer F.Cu)
-    (at 17.78 25.908)
+    (at 20.574 29.972)
     (descr "Diode SMA")
     (tags "Diode SMA")
     (attr smd)
-    (fp_text reference D1 (at 0 -3.81) (layer F.SilkS)
+    (fp_text reference D1 (at 0 -2.794) (layer F.SilkS)
       (effects (font (size 1 1) (thickness 0.15)))
     )
@@
   )
   (module Diodes_SMD:SMA_Standard (layer F.Cu)
-    (at 17.78 19.05)
+    (at 20.574 23.622)
     (descr "Diode SMA")
     (tags "Diode SMA")
     (attr smd)
-    (fp_text reference D2 (at 0 -3.81) (layer F.SilkS)
+    (fp_text reference D2 (at 0 -3.048) (layer F.SilkS)
       (effects (font (size 1 1) (thickness 0.15)))
     )
@@
     (tags "resistor 0805")
     (attr smd)
-    (fp_text reference R1 (at 0 2.1 90) (layer B.SilkS)
+    (fp_text reference R1 (at -3.81 -0.254 90) (layer B.SilkS)
       (effects (font (size 1 1) (thickness 0.15)) (justify mirror))
     )
-    (fp_text value 10K (at -2.794 2.032 90) (layer B.Fab)
+    (fp_text value 10K (at -4.064 0 90) (layer B.Fab) hide
       (effects (font (size 1 1) (thickness 0.15)) (justify mirror))
     )
@@
   )
   (module Resistors_SMD:R_0805_HandSoldering (layer F.Cu)
-    (at 26.416 18.796)
+    (at 28.702 24.384)
     (descr "Resistor SMD 0805, hand soldering")
     (tags "resistor 0805")
@@
     (descr "16x2 LCD footprint qith 16 pins")
     (tags "pin header")
-    (fp_text reference U1 (at 15.113 -7.0866 90) (layer F.SilkS)
+    (fp_text reference U1 (at -2.286 -1.524 90) (layer F.SilkS)
       (effects (font (size 1 1) (thickness 0.15)))
     )
@@
     )
   )
-  (gr_text "Designed by:\nMax Redmond\nElectromancy" (at 30.988 20.066) (layer B.Mask)
+  (gr_line (start 60.96 81.788) (end 60.96 81.28) (angle 90) (layer Edge.Cuts) (width 0.15))
+  (gr_line (start 15.24 81.788) (end 60.96 81.788) (angle 90) (layer Edge.Cuts) (width 0.15))
+  (gr_line (start 15.24 18.796) (end 15.24 81.788) (angle 90) (layer Edge.Cuts) (width 0.15))
+  (gr_line (start 60.96 18.796) (end 15.24 18.796) (angle 90) (layer Edge.Cuts) (width 0.15))
+  (gr_line (start 60.96 81.28) (end 60.96 18.796) (angle 90) (layer Edge.Cuts) (width 0.15))
+  (gr_text "Designed by:\nMax Redmond\nElectromancy" (at 31.242 25.654) (layer B.Mask)
     (effects (font (size 1.5 1.5) (thickness 0.3)) (justify left mirror))
   )
-  (gr_text "FM tuner\nv.1\n" (at 37.338 16.51) (layer F.SilkS)
+  (gr_text "FM tuner\nv.1\n" (at 44.196 23.368) (layer F.SilkS)
     (effects (font (size 1.5 1.5) (thickness 0.3)) (justify left))
   )
-  (gr_line (start 62.23 13.462) (end 62.23 13.208) (angle 90) (layer Edge.Cuts) (width 0.15))
   (gr_line (start 62.23 13.208) (end 62.23 13.462) (angle 90) (layer Edge.Cuts) (width 0.15))
-  (gr_line (start 13.208 13.208) (end 62.23 13.208) (angle 90) (layer Edge.Cuts) (width 0.15))
-  (gr_line (start 62.23 81.788) (end 13.208 81.788) (angle 90) (layer Edge.Cuts) (width 0.15))
-  (gr_line (start 13.208 81.788) (end 13.208 13.208) (angle 90) (layer Edge.Cuts) (width 0.15))
-  (gr_line (start 62.23 13.208) (end 62.23 81.788) (angle 90) (layer Edge.Cuts) (width 0.15))
   (segment (start -56.769 45.9232) (end -56.8452 45.9232) (width 0.25) (layer B.Cu) (net 0))
   (segment (start -61.849 45.9232) (end -61.849 46.101) (width 0.25) (layer B.Cu) (net 0))
   (segment (start -64.389 45.9232) (end -64.4652 45.9232) (width 0.25) (layer B.Cu) (net 0))
   (segment (start -54.229 45.9232) (end -54.229 45.847) (width 0.25) (layer B.Cu) (net 0))
-  (segment (start 34.778 28.956) (end 34.778 27.412) (width 0.25) (layer F.Cu) (net 2))
-  (segment (start 27.766 23.194) (end 29.464 24.892) (width 0.25) (layer F.Cu) (net 2))
-  (via (at 29.464 24.892) (size 0.6) (drill 0.4) (layers F.Cu B.Cu) (net 2))
-  (segment (start 27.766 23.194) (end 27.766 18.796) (width 0.25) (layer F.Cu) (net 2))
-  (segment (start 32.258 24.892) (end 29.464 24.892) (width 0.25) (layer F.Cu) (net 2))
-  (segment (start 34.778 27.412) (end 32.258 24.892) (width 0.25) (layer F.Cu) (net 2))
+  (via (at 37.064 25.908) (size 0.6) (drill 0.4) (layers F.Cu B.Cu) (net 2))
+  (segment (start 37.064 25.908) (end 37.084 25.908) (width 0.25) (layer B.Cu) (net 2))
+  (via (at 33.274 26.162) (size 0.6) (drill 0.4) (layers F.Cu B.Cu) (net 2))
+  (segment (start 31.496 24.384) (end 33.02 25.908) (width 0.25) (layer F.Cu) (net 2))
+  (segment (start 31.496 24.384) (end 30.052 24.384) (width 0.25) (layer F.Cu) (net 2) (status 800000))
+  (segment (start 34.778 28.956) (end 34.778 27.666) (width 0.25) (layer F.Cu) (net 2) (status 400000))
+  (segment (start 33.274 26.162) (end 33.02 25.908) (width 0.25) (layer F.Cu) (net 2))
+  (segment (start 34.778 27.666) (end 33.274 26.162) (width 0.25) (layer F.Cu) (net 2))
+  (segment (start 22.64454 37.0531) (end 26.1311 37.0531) (width 0.25) (layer F.Cu) (net 2))
+  (via (at 26.162 37.084) (size 0.6) (drill 0.4) (layers F.Cu B.Cu) (net 2))
+  (segment (start 26.1311 37.0531) (end 26.162 37.084) (width 0.25) (layer F.Cu) (net 2))
   (segment (start 34.116 65.024) (end 34.116 66.12) (width 0.25) (layer F.Cu) (net 2))
   (via (at 35.814 67.818) (size 0.6) (drill 0.4) (layers F.Cu B.Cu) (net 2))
@@
   (segment (start 43.757002 56.515) (end 57.2008 56.515) (width 0.25) (layer F.Cu) (net 2))
   (segment (start 42.360002 55.118) (end 43.757002 56.515) (width 0.25) (layer F.Cu) (net 2))
-  (segment (start 19.34254 37.5611) (end 25.6231 37.5611) (width 0.25) (layer F.Cu) (net 2))
-  (via (at 25.654 37.592) (size 0.6) (drill 0.4) (layers F.Cu B.Cu) (net 2))
-  (segment (start 25.6231 37.5611) (end 25.654 37.592) (width 0.25) (layer F.Cu) (net 2))
-  (segment (start 27.766 18.796) (end 34.29 18.796) (width 0.25) (layer F.Cu) (net 2))
-  (segment (start 34.29 18.796) (end 37.064 21.57) (width 0.25) (layer F.Cu) (net 2))
-  (segment (start 37.064 21.57) (end 37.064 23.622) (width 0.25) (layer F.Cu) (net 2))
-  (segment (start 37.064 23.622) (end 37.064 34.720314) (width 0.25) (layer F.Cu) (net 2))
+  (segment (start 37.064 23.622) (end 37.064 25.908) (width 0.25) (layer F.Cu) (net 2))
+  (segment (start 37.064 25.908) (end 37.064 27.94) (width 0.25) (layer F.Cu) (net 2))
+  (segment (start 37.064 27.94) (end 37.064 34.720314) (width 0.25) (layer F.Cu) (net 2))
   (segment (start 37.064 34.720314) (end 37.917639 35.573953) (width 0.25) (layer F.Cu) (net 2))
   (segment (start 34.778 28.956) (end 34.778 34.697056) (width 0.25) (layer F.Cu) (net 2))
@@
   (segment (start 57.2008 53.975) (end 45.085 53.975) (width 0.25) (layer F.Cu) (net 30))
   (segment (start 45.085 53.975) (end 44.958 53.848) (width 0.25) (layer F.Cu) (net 30))
+  (segment (start 28.622 35.306) (end 28.622 32.686) (width 0.25) (layer F.Cu) (net 42) (status 400000))
+  (segment (start 25.908 29.972) (end 22.57298 29.972) (width 0.25) (layer F.Cu) (net 42) (status 800000))
+  (segment (start 28.622 32.686) (end 25.908 29.972) (width 0.25) (layer F.Cu) (net 42))
   (segment (start 28.622 35.306) (end 28.622 34.75102) (width 0.25) (layer F.Cu) (net 42))
-  (segment (start 28.622 34.75102) (end 19.77898 25.908) (width 0.25) (layer F.Cu) (net 42))
-  (segment (start 20.28698 26.416) (end 19.77898 25.908) (width 0.25) (layer F.Cu) (net 42))
-  (segment (start 25.066 18.796) (end 20.03298 18.796) (width 0.25) (layer F.Cu) (net 43))
-  (segment (start 20.03298 18.796) (end 19.77898 19.05) (width 0.25) (layer F.Cu) (net 43))
+  (segment (start 27.352 24.384) (end 23.33498 24.384) (width 0.25) (layer F.Cu) (net 43) (status C00000))
+  (segment (start 23.33498 24.384) (end 22.57298 23.622) (width 0.25) (layer F.Cu) (net 43) (status C00000))
   (zone (net 1) (net_name GND) (layer F.Cu) (hatch edge 0.508)
     (connect_pads (clearance 0.3048))
@@
     (polygon
       (pts
-        (xy 62.23 81.788) (xy 13.208 81.788) (xy 13.208 13.208) (xy 62.23 13.208) (xy 62.23 81.788)
+        (xy 60.96 81.788) (xy 15.24 81.788) (xy 15.24 18.796) (xy 60.96 18.796) (xy 60.96 81.788)
       )
     )
-  )
-  (zone (net 2) (net_name VCC) (layer B.Cu) (hatch edge 0.508)
-    (connect_pads (clearance 0.508))
-    (min_thickness 0.254)
-    (fill yes (arc_segments 16) (thermal_gap 0.508) (thermal_bridge_width 0.508))
-    (polygon
-      (pts
-        (xy 62.23 81.788) (xy 13.208 81.788) (xy 13.208 13.208) (xy 62.23 13.208) (xy 62.23 81.788)
-      )
-    )
